File: pnp55te.kicad_pcb (KiCad board)
At the start: 2 copper layers, 154 x 109 mm, 68 parts, among them P1 1123038-2, U1 VNLD5090, U2 VNLD5090, U3 molex_48pin_MRE, U4 ITEAD_HC-05

Commit message: PNP adapter V0.1
Parts:
- removed D1, D2, D5, D6: D_Schottky, Diode_SMD:D_SMF
- removed D3, D4, D7, D8: LED, LED_SMD:LED_0603_1608Metric
- removed P1: 1123038-2, rusefi_pretty:1123038-2
- removed R10, R9: 10k, Resistor_SMD:R_0603_1608Metric
- removed R11, R12: 1k, Resistor_SMD:R_0603_1608Metric
- removed U2: VNLD5090, Package_SO:SO-8_3.9x4.9mm_P1.27mm
- removed U4: ITEAD_HC-05, rusEFI_Modules:ITEAD_HC-05
- removed W1, W10, W12, W13, W14, W19, W2, W24, W27, W28, W3, W30, W37, W5, W7, W9: TestPoint_2Pole, rusEFI_Modules:SM0805_jumper
- added BT1: Battery_Cell, rusEFI_Modules:BATT_CR2032_MPD, F.Cu at (161.2, 113.1)
- added H1: MountingHole_Pad, MountingHole:MountingHole_4mm_Pad_Via, F.Cu at (27.0, 95.0)
- added H2: MountingHole_Pad, MountingHole:MountingHole_4mm_Pad_Via, F.Cu at (54.5, 140.0)
- added H3: MountingHole_Pad, MountingHole:MountingHole_4mm_Pad_Via, F.Cu at (173.0, 95.0)
- added H4: MountingHole_Pad, MountingHole:MountingHole_4mm_Pad_Via, F.Cu at (145.5, 140.0)
- added TP1: TestPoint, TestPoint:TestPoint_THTPad_2.0x2.0mm_Drill1.0mm, F.Cu at (43.9, 103.2)
- added W38: TestPoint_2Pole, rusEFI_Modules:SM0805_jumper, F.Cu at (57.5, 60.4)
- added W39: TestPoint_2Pole, rusEFI_Modules:SM0805_jumper, F.Cu at (62.5, 60.4)
- added W40: TestPoint_2Pole, rusEFI_Modules:SM0805_jumper, F.Cu at (67.5, 60.4)
- added W40A1: TestPoint_2Pole, rusEFI_Modules:SM0805_jumper, B.Cu at (65.2, 76.7)
- added W41: TestPoint_2Pole, rusEFI_Modules:SM0805_jumper, F.Cu at (72.5, 60.4)
- added W42: TestPoint_2Pole, rusEFI_Modules:SM0805_jumper, F.Cu at (77.5, 60.4)
- added W42A1: TestPoint_2Pole, rusEFI_Modules:SM0805_jumper, B.Cu at (62.9, 76.6)
- added W44: TestPoint_2Pole, rusEFI_Modules:SM0805_jumper, F.Cu at (87.5, 60.4)
- added W46: TestPoint_2Pole, rusEFI_Modules:SM0805_jumper, F.Cu at (97.5, 60.4)
- added W47: TestPoint_2Pole, rusEFI_Modules:SM0805_jumper, F.Cu at (102.5, 60.4)
- added W48: TestPoint_2Pole, rusEFI_Modules:SM0805_jumper, F.Cu at (107.5, 60.4)
- added W49: TestPoint_2Pole, rusEFI_Modules:SM0805_jumper, F.Cu at (112.5, 60.4)
- added W50: TestPoint_2Pole, rusEFI_Modules:SM0805_jumper, F.Cu at (117.5, 60.4)
- added W51: TestPoint_2Pole, rusEFI_Modules:SM0805_jumper, F.Cu at (120.0, 60.4)
- added W54: TestPoint_2Pole, rusEFI_Modules:SM0805_jumper, F.Cu at (137.5, 60.4)
- added X1: 55pin_january_5.1, hw_55_te:TE_963063-2, F.Cu at (100.0, 40.0)
- C1: value 6.8n -> 100nF
- C2: value 6.8n -> 4.7uF; footprint Capacitor_SMD:C_0603_1608Metric -> Capacitor_SMD:C_0805_2012Metric
- C3, C4: value 6.8n -> 3.3nF
- C5: value 0.1u -> 100nF; footprint Capacitor_SMD:C_0805_2012Metric -> Capacitor_SMD:C_0603_1608Metric
- C6: value 1u -> 100nF; footprint Capacitor_SMD:C_0805_2012Metric -> Capacitor_SMD:C_0603_1608Metric
- R1, R2, R5, R6, R7, R8: value 1k -> R
- R3, R4: value 10k -> R
- U1: value VNLD5090 -> TPIC8101; footprint Package_SO:SO-8_3.9x4.9mm_P1.27mm -> Package_SO:SOIC-20W_7.5x12.8mm_P1.27mm
- U3: footprint rusEFI_Modules:Molex_48_MRE_with-extras -> hw_55_te:Molex_48_MRE_clean
- moved W4 225.9 mm to (70.0, 60.4), turned to 270 degrees
- moved W8 213.1 mm to (90.0, 60.4)
- moved C3 185.4 mm to (33.6, 103.1), turned to 90 degrees
- moved W15 183.7 mm to (125.0, 60.4), turned to 270 degrees
- moved C4 182.4 mm to (40.4, 103.8), turned to 225 degrees
- moved R8 177.8 mm to (43.8, 124.3), turned to 0 degrees
- moved C5 176.0 mm to (30.3, 116.4), turned to 180 degrees
- moved R7 174.5 mm to (43.8, 122.7), turned to 180 degrees
- moved C2 168.3 mm to (33.4, 124.6)
- moved C6 167.7 mm to (37.5, 122.7), turned to 0 degrees
- moved C1 164.8 mm to (33.4, 122.7)
- moved R4 164.4 mm to (37.7, 108.9)
- moved R1 162.0 mm to (33.6, 106.5), turned to 90 degrees
- moved R6 161.0 mm to (43.9, 107.2)
- moved R2 160.3 mm to (38.5, 106.5), turned to 90 degrees
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Connections:
- net /3L renamed Net-(W32-Pad2)
- net /3O renamed Net-(W18-Pad2)
- C1 pad 1: /LowSide1/OUT1 -> /MRE_5V
- C1 pad 2: GND -> /MRE_GND
- C2 pad 1: /LowSide1/OUT2 -> /MRE_5V
- C2 pad 2: GND -> /MRE_GND
- C3 pad 1: /LowSide2/OUT1 -> Net-(C3-Pad1)
- C3 pad 2: GND -> /KNOCK_IN
- C4 pad 1: /LowSide2/OUT2 -> Net-(C4-Pad1)
- C4 pad 2: GND -> Net-(C4-Pad2)
- C5 pad 1: GND -> Net-(C5-Pad1)
- C5 pad 2: /3v3 -> /MRE_GND
- C6 pad 1: /3v3 -> Net-(C6-Pad1)
- C6 pad 2: GND -> /MRE_GND
- R1 pad 2: /LowSide1/IN1 -> Net-(C3-Pad1)
- R2 pad 2: /LowSide1/IN2 -> Net-(C4-Pad2)
- R3 pad 1: Net-(R1-Pad1) -> Net-(R3-Pad1)
- R3 pad 2: GND -> Net-(R1-Pad1)
- R4 pad 1: Net-(R2-Pad1) -> Net-(R4-Pad1)
- R4 pad 2: GND -> Net-(R2-Pad1)
- R5 pad 1: Net-(D3-Pad2) -> /MRE_5V
- R5 pad 2: +12V -> /PC12_SPI3MOSI
- R6 pad 1: +12V -> /MRE_5V
- R6 pad 2: Net-(D4-Pad2) -> /PC10_SPI3SCK
- R7 pad 1: Net-(R7-Pad1) -> /MRE_5V
- R7 pad 2: /LowSide2/IN1 -> /PA15_SPI3CS
- R8 pad 1: Net-(R10-Pad1) -> /PB9
- R8 pad 2: /LowSide2/IN2 -> /MRE_5V
- U1 pad 1: Net-(R1-Pad1) -> /MRE_5V
- U1 pad 2: Net-(U1-Pad2) -> /MRE_GND
- U1 pad 3: Net-(R2-Pad1) -> Net-(C5-Pad1)
- U1 pad 4: Net-(U1-Pad4) -> Net-(C6-Pad1)
- U1 pad 5: GND -> (no net)
- U1 pad 6: /LowSide1/OUT2 -> (no net)
- U1 pad 7: GND -> /PB9
- U1 pad 8: /LowSide1/OUT1 -> /PA15_SPI3CS
- U3 pad 1: Net-(U3-Pad1) -> /12_MAIN_RELAY
- U3 pad 10: Net-(U3-Pad10) -> /HI2_UNUSED
- U3 pad 11: Net-(U3-Pad11) -> /COIL2
- U3 pad 12: Net-(U3-Pad12) -> /HI4_UNUSED
- U3 pad 13: Net-(U3-Pad13) -> /ECO_OUT
- U3 pad 14: Net-(U3-Pad14) -> /TACH
- U3 pad 15: Net-(U3-Pad15) -> (no net)
- U3 pad 16: Net-(U3-Pad16) -> (no net)
- U3 pad 17: Net-(U3-Pad17) -> /GND_SENS_1
- U3 pad 18: Net-(U3-Pad18) -> /CLT
- U3 pad 19: Net-(U3-Pad19) -> /STEERING_REQ
- U3 pad 2: Net-(U3-Pad2) -> GND
- U3 pad 20: Net-(U3-Pad20) -> /EGR_POS
- U3 pad 21: Net-(U3-Pad21) -> /GND_SENS_2
- U3 pad 22: Net-(U3-Pad22) -> /RESERVED_AIN1
- U3 pad 23: Net-(U3-Pad23) -> /IAT
- U3 pad 24: Net-(U3-Pad24) -> /RESERVED_AIN2
- U3 pad 25: Net-(U3-Pad25) -> /CAM_HALL
- U3 pad 26: Net-(U3-Pad26) -> /TPS
- U3 pad 27: Net-(U3-Pad27) -> /MAF
- U3 pad 28: Net-(U3-Pad28) -> /L_LINE
- U3 pad 29: Net-(U3-Pad29) -> /MAIN_RELAY_CONTROL
- U3 pad 3: Net-(U3-Pad3) -> /AFR_HEATER
- U3 pad 30: Net-(U3-Pad30) -> /AC_RELAY
- U3 pad 31: Net-(U3-Pad31) -> /ABSORBER_VALVE
- U3 pad 32: Net-(U3-Pad32) -> /AFR_NARROW
- U3 pad 33: Net-(U3-Pad33) -> /IDLE_STEP_C
- U3 pad 34: Net-(U3-Pad34) -> /IDLE_STEP_B
- U3 pad 35: Net-(U3-Pad35) -> /IDLE_STEP_A
- U3 pad 36: Net-(U3-Pad36) -> /AC_REQUEST
- U3 pad 37: Net-(U3-Pad37) -> /INJ1
- U3 pad 38: Net-(U3-Pad38) -> /INJ2
- U3 pad 39: Net-(U3-Pad39) -> /5V_SENS2
- U3 pad 4: Net-(U3-Pad4) -> (no net)
- U3 pad 40: Net-(U3-Pad40) -> /RESERVED_AIN0
- U3 pad 41: Net-(U3-Pad41) -> /INJ3
- U3 pad 42: Net-(U3-Pad42) -> /INJ4
- U3 pad 43: Net-(U3-Pad43) -> /IDLE_STEP_D
- U3 pad 44: Net-(U3-Pad44) -> (no net)
- U3 pad 45: Net-(U3-Pad45) -> /CRANK_p
- U3 pad 46: Net-(U3-Pad46) -> /CRANK_n
- U3 pad 47: Net-(U3-Pad47) -> /CAN_L
- U3 pad 48: Net-(U3-Pad48) -> /CAN_H
- U3 pad 5: Net-(U3-Pad5) -> /12_IGN_KEY
- U3 pad 6: Net-(U3-Pad6) -> GND
- U3 pad 7: Net-(U3-Pad7) -> /RESERVED_HI_CUR
- U3 pad 8: Net-(U3-Pad8) -> (no net)
- U3 pad 9: Net-(U3-Pad9) -> /COIL1
- U3 pad J31: Net-(U3-PadJ31) -> /VBAT
- U3 pad J61: Net-(U3-PadJ61) -> /FUEL_RELAY
- U3 pad J62: Net-(U3-PadJ62) -> /MIL
- U3 pad J63: Net-(U3-PadJ63) -> /FAN_RELAY
- U3 pad J64: Net-(U3-PadJ64) -> /EGR_VALVE
- U3 pad J65: Net-(U3-PadJ65) -> /VAR_INTAKE
- U3 pad J801: Net-(U3-PadJ801) -> /MRE_5V
- U3 pad J802: Net-(U3-PadJ802) -> (no net)
- U3 pad J803: Net-(U3-PadJ803) -> (no net)
- U3 pad J804: Net-(U3-PadJ804) -> (no net)
- U3 pad J805: Net-(U3-PadJ805) -> /PC11_SPI3MISO
- U3 pad J806: Net-(U3-PadJ806) -> /PB9
- U3 pad J807: Net-(U3-PadJ807) -> /PA15_SPI3CS
- U3 pad J808: Net-(U3-PadJ808) -> /PC10_SPI3SCK
- U3 pad J809: Net-(U3-PadJ809) -> /MRE_GND
- U3 pad J810: Net-(U3-PadJ810) -> /PC12_SPI3MOSI
- U3 pad LIN1: Net-(U3-PadLIN1) -> /LIN
- U3 pad M11: Net-(U3-PadM11) -> (no net)
- U3 pad M12: Net-(U3-PadM12) -> (no net)
- U3 pad M13: Net-(U3-PadM13) -> (no net)
- U3 pad M21: Net-(U3-PadM21) -> (no net)
- U3 pad M22: Net-(U3-PadM22) -> (no net)
- U3 pad M23: Net-(U3-PadM23) -> (no net)
- U3 pad M3: Net-(U3-PadM3) -> (no net)
- U3 pad M4: Net-(U3-PadM4) -> (no net)
- U3 pad M51: Net-(U3-PadM51) -> (no net)
- U3 pad M52: Net-(U3-PadM52) -> (no net)
- U3 pad M53: Net-(U3-PadM53) -> (no net)
- U3 pad M61: Net-(U3-PadM61) -> (no net)
- U3 pad M62: Net-(U3-PadM62) -> (no net)
- U3 pad M63: Net-(U3-PadM63) -> (no net)
- U3 pad M71: Net-(U3-PadM71) -> (no net)
- U3 pad M72: Net-(U3-PadM72) -> (no net)
- U3 pad M73: Net-(U3-PadM73) -> (no net)
- W11 pad 1: /VVT -> Net-(W11-Pad1)
- W11 pad 2: /4R -> /KNOCK_IN
- W15 pad 1: /COIL1 -> Net-(W15-Pad1)
- W15 pad 2: /3F -> /AFR_HEATER
- W16 pad 1: /COIL2 -> Net-(W16-Pad1)
- W16 pad 2: /3I -> /INJ2
- W17 pad 1: /ALTERNATOR -> Net-(W17-Pad1)
- W17 pad 2: /3M -> /EGR_VALVE
- W18 pad 1: /TACH -> Net-(W18-Pad1)
- W20 pad 1: /5V_SENS1 -> Net-(W20-Pad1)
- W20 pad 2: /4L -> /COIL2
- W21 pad 1: /GND_SENS -> Net-(W21-Pad1)
- W21 pad 2: /4O -> /IDLE_STEP_C
- W22 pad 1: /ALT_WARN -> Net-(W22-Pad1)
- W22 pad 2: /VNLSD5160_from_PB8 -> /MIL
- W23 pad 1: /5V_SENS2 -> Net-(W23-Pad1)
- W23 pad 2: /4G -> /INJ1
- W25 pad 1: /GND_SENS -> Net-(W25-Pad1)
- W25 pad 2: /4G -> /AC_RELAY
- W26 pad 1: /AFR -> Net-(W26-Pad1)
- W26 pad 2: /4Q -> /IDLE_STEP_B
- W29 pad 1: /TPS -> Net-(W29-Pad1)
- W29 pad 2: /4V -> /IDLE_STEP_D
- W31 pad 1: /CRANK -> Net-(W31-Pad1)
- W31 pad 2: /3Y -> /RESERVED_HI_CUR
- W32 pad 1: /CAN_H -> Net-(W32-Pad1)
- W33 pad 1: /CAN_L -> Net-(W33-Pad1)
- W33 pad 2: /3N -> /AFR_HEATER
- W34 pad 1: /USBD- -> Net-(W34-Pad1)
- W34 pad 2: /3W -> /INJ4
- W35 pad 1: /USBD+ -> Net-(W35-Pad1)
- W35 pad 2: /3X -> /INJ3
- W36 pad 1: /USB_GND -> Net-(W36-Pad1)
- W36 pad 2: /3Z -> /VAR_INTAKE
- W4 pad 1: /INJ4 -> Net-(W4-Pad1)
- W4 pad 2: /2J -> /IDLE_STEP_A
- W6 pad 1: /MAIN_RELAY_CONTROL -> Net-(W6-Pad1)
- W6 pad 2: /3H -> /FAN_RELAY
- W8 pad 1: /12_MAIN_RELAY -> Net-(W8-Pad1)
- W8 pad 2: /4D -> /CAM_HALL
Routing:
- net GND: track 0.00 -> 340.7 mm
- net /12_MAIN_RELAY: track 0.00 -> 139.9 mm
- net /GND_SENS_2: track 0.00 -> 117.3 mm
- net /5V_SENS2: track 0.00 -> 116.2 mm, vias 0 -> 1
- net /MRE_5V: track 0.00 -> 114.1 mm, vias 0 -> 4
- net /GND_SENS_1: track 0.00 -> 113.7 mm
- net /ECO_OUT: track 0.00 -> 108.6 mm, vias 0 -> 1
- net /INJ2: track 0.00 -> 107.8 mm, vias 0 -> 1
- net /KNOCK_IN: track 0.00 -> 106.0 mm, vias 0 -> 1
- net /INJ3: track 0.00 -> 103.3 mm, vias 0 -> 1
- net /TPS: track 0.00 -> 103.1 mm, vias 0 -> 1
- net /AFR_HEATER: track 0.00 -> 101.9 mm
- net /INJ4: track 0.00 -> 99.6 mm, vias 0 -> 1
- net /RESERVED_AIN2: track 0.00 -> 95.8 mm, vias 0 -> 1
- net /12_IGN_KEY: track 0.00 -> 95.8 mm
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- added copper zone on B.Cu, net /MRE_GND
- removed copper zone on F.Cu, net GND
Other:
- outline, holes or cut-outs redrawn
- board text removed: "TODO: 4 vertical signal vias just in case"
- board text removed: "TODO: 5 vertical signal vias"
- board text removed: "TODO: J4.J8 vias 2x5"
- board text removed: "bluetooth footprint from Frankenso"
